Commit message: New Assembly

File: ros_noetic_catkin_ws/src/robot_arm_urdf/urdf/robot_arm_urdf.urdf (robot description, URDF)
Before this commit: robot robot_arm_urdf, 7 links, 6 joints
Links:
- link base_link: mass 2.27847589927695 -> 1.2708
- link link_1: mass 0.641883744293896 -> 0.10142
- link link_2: mass 0.394669428659782 -> 0.39467
- link link_3: mass 0.259256412516919 -> 0.25926
- link link_4: mass 0.18731544221453 -> 0.18732
- link link_5: mass 0.00352439273827263 -> 0.0035244
Joints:
- joint joint_1: axis 0 1 0 -> 0 0 1; origin xyz=0.004244 0.37679 -0.077856 rpy=1.5708 0 0 -> xyz=0 0 0.15678 rpy=0 0 0
- joint joint_2: axis -0.125391445630158 0 -0.992107345685324 -> -0.12539 0.99211 0; origin xyz=-0.0129136150732728 0.308337646724069 0.307358400547654 rpy=0 0 0 -> xyz=0.00010358 1.3092E-05 0.0737 rpy=0 0 0
- joint joint_3: axis -0.125391445630158 0 -0.992107345685324 -> 0.12539 -0.99211 0; origin xyz=-0.0040937973882068 0.406399999999999 -0.0323904588559681 rpy=0 0 0 -> xyz=0 0 0.4064 rpy=0 0 0
- joint joint_4: axis -0.125391445630158 0 -0.992107345685324 -> -0.12539 0.99211 0; origin xyz=-0.344415980373364 0 0.0713450468234001 rpy=0 0 0 -> xyz=-0.34841 -0.039718 0 rpy=0 0 0
- joint joint_5: axis 0 -1 0 -> 0 0 -1; origin xyz=0.00886960764909822 0.0715224872569122 0.0701770591910485 rpy=0 0 0 -> xyz=0 0 0.077198 rpy=0 0 0

Commit message: Added moveit package without EE.

File: ros_noetic_catkin_ws/src/robot_arm_urdf/urdf/robot_arm_urdf.urdf (robot description, URDF)
Before this commit: robot robot_arm_urdf, 7 links, 6 joints
Joints:
- joint joint_3: limit lower=-1 upper=3.14 effort=7.85 velocity=6.54 -> lower=-3.14 upper=1 effort=7.85 velocity=6.54
