Commit message: updated solidworks model correctly

File: full_assembly2_urdf/urdf/full_assembly2_urdf.urdf (robot description, URDF)
Before this commit: robot full_robot_arm_urdf, 14 links, 13 joints
Links:
- link base_link: mass 1.2708 -> 1.2708035851133; geometry collision mesh filename=package://full_assembly2_urdf/meshes/base_link.STL; visual mesh filename=package://full_assembly2_urdf/meshes/base_link.STL
- link ee_finger1_dist: mass 0.01344 -> 0.0134397344943946; geometry collision mesh filename=package://full_assembly2_urdf/meshes/ee_finger1_dist.STL; visual mesh filename=package://full_assembly2_urdf/meshes/ee_finger1_dist.STL
- link ee_finger1_prox: mass 0.0146611614005227 -> 0.0145193149160156; geometry collision mesh filename=package://full_assembly2_urdf/meshes/ee_finger1_prox.STL; visual mesh filename=package://full_assembly2_urdf/meshes/ee_finger1_prox.STL
- link ee_finger1_roll: mass 0.026092694642213 -> 0.0130633836142709; geometry collision mesh filename=package://full_assembly2_urdf/meshes/ee_finger1_roll.STL; visual mesh filename=package://full_assembly2_urdf/meshes/ee_finger1_roll.STL
- link ee_finger2_dist: mass 0.013599 -> 0.01344001329834; geometry collision mesh filename=package://full_assembly2_urdf/meshes/ee_finger2_dist.STL; visual mesh filename=package://full_assembly2_urdf/meshes/ee_finger2_dist.STL
- link ee_finger2_prox: mass 0.0146611931889972 -> 0.014519343110467; geometry collision mesh filename=package://full_assembly2_urdf/meshes/ee_finger2_prox.STL; visual mesh filename=package://full_assembly2_urdf/meshes/ee_finger2_prox.STL
- link ee_finger2_roll: mass 0.0232082046067633 -> 0.0130633776120231; geometry collision mesh filename=package://full_assembly2_urdf/meshes/ee_finger2_roll.STL; visual mesh filename=package://full_assembly2_urdf/meshes/ee_finger2_roll.STL
- link ee_thumb_dist: mass 0.011962 -> 0.0116864486254284; geometry collision mesh filename=package://full_assembly2_urdf/meshes/ee_thumb_dist.STL; visual mesh filename=package://full_assembly2_urdf/meshes/ee_thumb_dist.STL
- link ee_thumb_prox: geometry collision mesh filename=package://full_assembly2_urdf/meshes/ee_thumb_prox.STL; visual mesh filename=package://full_assembly2_urdf/meshes/ee_thumb_prox.STL
- link link_1: mass 0.64188 -> 0.641883793391617; geometry collision mesh filename=package://full_assembly2_urdf/meshes/link_1.STL; visual mesh filename=package://full_assembly2_urdf/meshes/link_1.STL
- link link_2: mass 0.39695 -> 0.394669414155339; geometry collision mesh filename=package://full_assembly2_urdf/meshes/link_2.STL; visual mesh filename=package://full_assembly2_urdf/meshes/link_2.STL
- link link_3: mass 0.271185231914755 -> 0.259256414102; geometry collision mesh filename=package://full_assembly2_urdf/meshes/link_3.STL; visual mesh filename=package://full_assembly2_urdf/meshes/link_3.STL
- link link_4: mass 0.18731544179836 -> 0.187315441798361; geometry collision mesh filename=package://full_assembly2_urdf/meshes/link_4.STL; visual mesh filename=package://full_assembly2_urdf/meshes/link_4.STL
- link link_5: mass 0.451187361366382 -> 0.183111513613456; geometry collision mesh filename=package://full_assembly2_urdf/meshes/link_5.STL; visual mesh filename=package://full_assembly2_urdf/meshes/link_5.STL
Joints:
- joint ee_finger1_dist_joint: axis -0.69373 -0.72024 0 -> -0.693726536855436 -0.720238496654104 0; origin xyz=-0.025475 0.024538 0.03534 rpy=0 0 0 -> xyz=-0.0254754976779759 0.0245377452898056 0.0353397520386329 rpy=0 0 0
- joint ee_finger1_prox_joint: axis -0.69373 -0.72024 0 -> -0.693726536855436 -0.720238496654104 0; origin xyz=0 0 0.043 rpy=0 0 0 -> xyz=0 0 0.0430000000000001 rpy=0 0 0
- joint ee_finger1_roll_joint: origin xyz=-0.02203 -0.029016 0.039425 rpy=0 0 1.6777 -> xyz=-0.0220304161455278 -0.0290156985863783 0.039424999999998 rpy=0 0 1.67767623706565
- joint ee_finger2_dist_joint: axis 0.70063 -0.71353 0 -> 0.700628532140015 -0.713526215321714 0; origin xyz=0.024968 0.024516 0.035715 rpy=0 0 0 -> xyz=0.0249677805106804 0.0245164634940634 0.0357148842097346 rpy=0 0 0
- joint ee_finger2_prox_joint: axis 0.70063 -0.71353 0 -> 0.700628532140014 -0.713526215321714 0; origin xyz=-4.8612E-05 4.9507E-05 0.043 rpy=0 0 0 -> xyz=-4.86118565775811E-05 4.95067392380366E-05 0.0429999999999999 rpy=0 0 0
- joint ee_finger2_roll_joint: origin xyz=-0.028004 0.026665 0.039425 rpy=0 0 1.6777 -> xyz=-0.0280043023470612 0.0266647529531982 0.0394249999999982 rpy=0 0 1.67767623706565
- joint ee_thumb_dist_joint: origin xyz=0 -0.035355 0.035355 rpy=0 0 0 -> xyz=0 -0.035355339059327 0.0353553390593278 rpy=0 0 0
- joint ee_thumb_prox_joint: origin xyz=0.044583 0.0062919 0.080425 rpy=0 0 1.6777 -> xyz=0.0445832051781762 0.00629188493532656 0.0804249999999981 rpy=0 0 1.67767623706565
- joint joint_2: axis -0.12539 0.99211 0 -> -0.125391445630158 0.992107345685324 0; origin xyz=0.00010358 1.3092E-05 0.0737 rpy=0 0 0 -> xyz=0.000103583713295205 1.30918409286529E-05 0.0737000000000103 rpy=0 0 0
- joint joint_3: axis 0.12539 -0.99211 0 -> 0.125391445630158 -0.992107345685324 0; origin xyz=0 0 0.4064 rpy=0 0 0 -> xyz=0 0 0.406399999999993 rpy=0 0 0
- joint joint_4: axis -0.12539 0.99211 0 -> -0.125391445630158 0.992107345685324 0; origin xyz=-0.34841 -0.039718 0 rpy=0 0 0 -> xyz=-0.348413326699186 -0.0397177166403455 0 rpy=0 0 0
- joint joint_5: origin xyz=0 0 0.077198 rpy=0 0 0 -> xyz=0 0 0.0771975122568782 rpy=0 0 0
