Commit message: another test

File: ros_noetic_catkin_ws/src/full_robot_arm_urdf/urdf/full_robot_arm_urdf.urdf (robot description, URDF)
Before this commit: robot full_robot_arm_urdf, 15 links, 14 joints
Links:
- link base_link: mass 1.2708035851133 -> 1.2708
- link link_4: mass 0.187315441798361 -> 0.18731544179836
Joints:
- joint ee_finger1_dist_joint: axis -0.693726536855436 -0.720238496654104 0 -> -1 0 0; origin xyz=-0.0254754976779759 0.0245377452898056 0.0353397520386329 rpy=0 0 0 -> xyz=0 0.042932 -0.0070742 rpy=0.005151 0 0
- joint ee_finger1_prox_joint: axis -0.693726536855436 -0.720238496654104 0 -> -1 0 0; origin xyz=0 0 0.0430000000000001 rpy=0 0 0 -> xyz=0 0.01 0 rpy=-0.78584 0 0
- joint ee_finger1_roll_joint: axis 0 0 -1 -> 0 -1 0; origin xyz=-0.0220304161455278 -0.0290156985863783 0.039424999999998 rpy=0 0 1.67767623706565 -> xyz=-0.053886 -0.063523 0.027809 rpy=-3.1416 -0.83742 0
- joint ee_finger2_dist_joint: axis 0.700628532140015 -0.713526215321714 0 -> -1 0 0; origin xyz=0.0249677805106804 0.0245164634940634 0.0357148842097346 rpy=0 0 0 -> xyz=6.9383E-05 0.042857 0.0069984 rpy=-0.012196 0 0
- joint ee_finger2_prox_joint: axis 0.700628532140014 -0.713526215321714 0 -> -1 0 0; origin xyz=-4.86118565775811E-05 4.95067392380366E-05 0.0429999999999999 rpy=0 0 0 -> xyz=0 0.01 0 rpy=0.77518 0 0
- joint ee_finger2_roll_joint: axis 0 0 -1 -> 0 -1 0; origin xyz=-0.0280043023470612 0.0266647529531982 0.0394249999999982 rpy=0 0 1.67767623706565 -> xyz=0.0020832 -0.063523 0.029672 rpy=0 -0.76125 3.1416
- joint ee_thumb_dist_joint: axis 1 0 0 -> -1 0 0; origin xyz=0 -0.035355339059327 0.0353553390593278 rpy=0 0 0 -> xyz=0 0.05 0 rpy=0 0 0
- joint ee_thumb_prox_joint: axis 1 0 0 -> -1 0 0; origin xyz=0.0445832051781762 0.00629188493532656 0.0804249999999981 rpy=0 0 1.67767623706565 -> xyz=-0.023573 -0.061523 -0.041221 rpy=-0.7854 0.033272 3.1416
- joint joint_1: axis 0 0 1 -> 0 1 0; origin xyz=0 0 0.1567815 rpy=0 0 0 -> xyz=-0.081165 -0.018898 0.39934 rpy=1.566 -0.01307 -0.7805
- joint joint_2: axis -0.125391445630158 0.992107345685324 0 -> 0 0 -1; origin xyz=0.000103583713295205 1.30918409286529E-05 0.0737000000000103 rpy=0 0 0 -> xyz=0.048155 0.06735 0.012605 rpy=0.77684 0 1.5708
- joint joint_3: axis 0.125391445630158 -0.992107345685324 0 -> 0 1 0; origin xyz=0 0 0.406399999999993 rpy=0 0 0 -> xyz=0.4064 0.0254 -0.080236 rpy=1.5708 0 -2.0944
- joint joint_4: axis -0.125391445630158 0.992107345685324 0 -> 0 0 1; origin xyz=-0.348413326699186 -0.0397177166403455 0 rpy=0 0 0 -> xyz=-0.30367 0.058389 0.17532 rpy=-1.5708 -0.9167 -3.1416
- joint joint_5: axis 0 0 -1 -> 0 1 0; origin xyz=0 0 0.0771975122568782 rpy=0 0 0 -> xyz=-0.041507 0.086823 0.051524 rpy=0 -1.5187 -2.7485

Commit message: Small changes to previous urdf

File: ros_noetic_catkin_ws/src/full_robot_arm_urdf/urdf/full_robot_arm_urdf.urdf (robot description, URDF)
Before this commit: robot full_robot_arm_urdf, 15 links, 14 joints
Links:
- link ee_finger1_dist: mass 0.0134397344943946 -> 0.0134397344943939
- link ee_finger1_prox: mass 0.0145193149160156 -> 0.0145193149160161
- link ee_finger1_roll: mass 0.0130633836142709 -> 0.0130633836142706
- link ee_finger2_dist: mass 0.01344001329834 -> 0.0134400132983415
- link ee_finger2_prox: mass 0.014519343110467 -> 0.0145193439812253
- link ee_thumb_prox: mass 0.0140616051661292 -> 0.0140616075473925
- link link_1: mass 0.641883793391617 -> 0.641883793389845
- link link_2: mass 0.394669414155339 -> 0.394669414176607
- link link_3: mass 0.259256414102 -> 0.259256414101999
- link link_5: mass 0.183111513613456 -> 0.183111545605538
Joints:
- joint ee_finger1_dist_joint: limit lower=0 upper=1.57 effort=2.45 velocity=8.08 -> lower=-1.57 upper=0 effort=2.45 velocity=8.08; origin xyz=0 0.042932 -0.0070742 rpy=0.005151 0 0 -> xyz=0.31567 0.10487 0.18973 rpy=0.79011 0 0.80415
- joint ee_finger1_prox_joint: axis -1 0 0 -> -0.69373 -0.72024 0; limit lower=0 upper=1.57 effort=2.45 velocity=8.08 -> lower=-1.57 upper=0 effort=2.45 velocity=8.08; origin xyz=0 0.01 0 rpy=-0.78584 0 0 -> xyz=-0.29452 -0.15439 -0.18998 rpy=-1.5708 -0.80415 0
- joint ee_finger1_roll_joint: origin xyz=-0.053886 -0.063523 0.027809 rpy=-3.1416 -0.83742 0 -> xyz=-0.138295266521999 0.301612506052774 0.236814827435665 rpy=1.57079632679489 0 2.48182228526102
- joint ee_finger2_dist_joint: origin xyz=6.9383E-05 0.042857 0.0069984 rpy=-0.012196 0 0 -> xyz=0.366112078928804 0.104847608094271 0.1901047116454 rpy=2.33377636483635 0 2.34707432452152
- joint ee_finger2_prox_joint: axis -1 0 0 -> 0.700628532140014 -0.713526215321714 0; origin xyz=0 0.01 0 rpy=0.77518 0 0 -> xyz=0.181766434679577 -0.154389827435665 -0.299697692055236 rpy=1.5707963267949 -0.794518329068275 -3.14159265358979
- joint ee_finger2_roll_joint: origin xyz=0.0020832 -0.063523 0.029672 rpy=0 -0.76125 3.1416 -> xyz=-0.144269152723533 0.357292957592351 0.236814827435665 rpy=1.57079632679489 0 -2.25843474559242
- joint ee_thumb_dist_joint: limit lower=0 upper=1.57 effort=2.45 velocity=8.08 -> lower=-1.57 upper=0 effort=2.45 velocity=8.08
- joint ee_thumb_prox_joint: limit lower=0 upper=1.57 effort=2.45 velocity=8.08 -> lower=-1.57 upper=0 effort=2.45 velocity=8.08; origin xyz=-0.023573 -0.061523 -0.041221 rpy=-0.7854 0.033272 3.1416 -> xyz=-0.071682 0.33692 0.23481 rpy=0.7854 0 -1.4639
- joint joint_1: axis 0 1 0 -> 0 0 1; origin xyz=-0.081165 -0.018898 0.39934 rpy=1.566 -0.01307 -0.7805 -> xyz=-0.0076079 -0.36376 0.24337 rpy=-0.011751 -0.0074781 -0.12937
- joint joint_2: axis 0 0 -1 -> -0.12539 0.99211 0; origin xyz=0.048155 0.06735 0.012605 rpy=0.77684 0 1.5708 -> xyz=0.00010358 1.3092E-05 0.0737 rpy=0 0 0
- joint joint_3: limit lower=-1 upper=3.14 effort=7.85 velocity=6.54 -> lower=-3.14 upper=1 effort=7.85 velocity=6.54; origin xyz=0.4064 0.0254 -0.080236 rpy=1.5708 0 -2.0944 -> xyz=-0.12097 0.36782 0.56079 rpy=-3.1416 0.5236 0.12572
- joint joint_5: axis 0 1 0 -> 0 0 -1; origin xyz=-0.041507 0.086823 0.051524 rpy=0 -1.5187 -2.7485 -> xyz=-0.038685 -0.099608 -0.31741 rpy=1.5708 0.12572 -2.7485

Commit message: testing again

File: ros_noetic_catkin_ws/src/full_robot_arm_urdf/urdf/full_robot_arm_urdf.urdf (robot description, URDF)
Before this commit: robot full_robot_arm_urdf, 15 links, 14 joints
Links:
- link ee_thumb_prox: mass 0.0140616075473925 -> 0.0140616075473926
- link link_1: mass 0.641883793389845 -> 0.641883793389852
Joints:
- joint ee_finger1_dist_joint: origin xyz=0.31567 0.10487 0.18973 rpy=0.79011 0 0.80415 -> xyz=-0.0054971 1.0558 0.23694 rpy=0.005151 0 0
- joint ee_finger1_prox_joint: axis -0.69373 -0.72024 0 -> -1 0 0; origin xyz=-0.29452 -0.15439 -0.18998 rpy=-1.5708 -0.80415 0 -> xyz=0.0054971 -0.87853 0.54407 rpy=-0.78584 0 0
- joint ee_finger1_roll_joint: origin xyz=-0.138295266521999 0.301612506052774 0.236814827435665 rpy=1.57079632679489 0 2.48182228526102 -> xyz=-0.053886 -0.063523 0.027809 rpy=-3.1416 -0.83742 0
- joint ee_finger2_dist_joint: origin xyz=0.366112078928804 0.104847608094271 0.1901047116454 rpy=2.33377636483635 0 2.34707432452152 -> xyz=6.9383E-05 0.05 0 rpy=-0.012196 0 0
- joint ee_finger2_prox_joint: axis 0.700628532140014 -0.713526215321714 0 -> -1 0 0; origin xyz=0.181766434679577 -0.154389827435665 -0.299697692055236 rpy=1.5707963267949 -0.794518329068275 -3.14159265358979 -> xyz=0 0 0 rpy=0.77518 0 0
- joint ee_finger2_roll_joint: origin xyz=-0.144269152723533 0.357292957592351 0.236814827435665 rpy=1.57079632679489 0 -2.25843474559242 -> xyz=0.0020832 -0.063523 0.029672 rpy=0 -0.76125 -3.1416
- joint ee_thumb_prox_joint: origin xyz=-0.071682 0.33692 0.23481 rpy=0.7854 0 -1.4639 -> xyz=-0.023573 -0.061523 -0.041221 rpy=-0.7854 0.033272 3.1416
- joint joint_1: axis 0 0 1 -> 0 1 0; origin xyz=-0.0076079 -0.36376 0.24337 rpy=-0.011751 -0.0074781 -0.12937 -> xyz=-0.0076454 -0.36368 0.24972 rpy=1.566 -0.01307 -0.7805
- joint joint_2: axis -0.12539 0.99211 0 -> 0 0 -1; origin xyz=0.00010358 1.3092E-05 0.0737 rpy=0 0 0 -> xyz=0.048155 0.06735 0.012605 rpy=0.77684 0 1.5708
- joint joint_3: origin xyz=-0.12097 0.36782 0.56079 rpy=-3.1416 0.5236 0.12572 -> xyz=0.4064 0.0254 -0.080236 rpy=1.5708 0 -2.0944
- joint joint_5: axis 0 0 -1 -> 0 1 0; origin xyz=-0.038685 -0.099608 -0.31741 rpy=1.5708 0.12572 -2.7485 -> xyz=-0.041507 0.086823 0.051524 rpy=0 -1.5187 -2.7485

Commit message: small origin changes

File: ros_noetic_catkin_ws/src/full_robot_arm_urdf/urdf/full_robot_arm_urdf.urdf (robot description, URDF)
Before this commit: robot full_robot_arm_urdf, 15 links, 14 joints
Links:
- link ee_thumb_prox: mass 0.0140616075473926 -> 0.0140616075473925
- link link_1: mass 0.641883793389852 -> 0.641883793389845
- link link_2: mass 0.394669414176607 -> 0.394669414176608
Joints:
- joint ee_finger1_dist_joint: origin xyz=-0.0054971 1.0558 0.23694 rpy=0.005151 0 0 -> xyz=0 0.05 0 rpy=0.0051509884381174 0 0
- joint ee_finger1_prox_joint: origin xyz=0.0054971 -0.87853 0.54407 rpy=-0.78584 0 0 -> xyz=0 0 0 rpy=-0.78584 0 0
- joint ee_finger1_roll_joint: origin xyz=-0.053886 -0.063523 0.027809 rpy=-3.1416 -0.83742 0 -> xyz=-0.0273169803327454 -0.082424999999998 0.0241046175141006 rpy=-3.14159265358979 -0.837418070437063 0
- joint ee_finger2_dist_joint: origin xyz=6.9383E-05 0.05 0 rpy=-0.012196 0 0 -> xyz=6.93832099998293E-05 0.0499999999999999 0 rpy=-0.0121962316875519 0 0
- joint ee_finger2_prox_joint: origin xyz=0 0 0 rpy=0.77518 0 0 -> xyz=0 0 0 rpy=0.775176269729007 0 0
- joint ee_finger2_roll_joint: origin xyz=0.0020832 -0.063523 0.029672 rpy=0 -0.76125 -3.1416 -> xyz=0.0286520257576785 -0.0824249999999981 0.0259675070036006 rpy=0 -0.761246306826586 -3.14159265358979
- joint ee_thumb_dist_joint: origin xyz=0 0.05 0 rpy=0 0 0 -> xyz=0 0.0500000000000002 0 rpy=0 0 0
- joint ee_thumb_prox_joint: origin xyz=-0.023573 -0.061523 -0.041221 rpy=-0.7854 0.033272 3.1416 -> xyz=0.00299613457434156 -0.0804249999999981 -0.0449251953541793 rpy=-0.785398163397437 0.0332720222416905 3.14159265358979
- joint joint_2: origin xyz=0.048155 0.06735 0.012605 rpy=0.77684 0 1.5708 -> xyz=7.4457E-05 0.06735 -7.3193E-05 rpy=0.77684 0 1.5708
- joint joint_3: origin xyz=0.4064 0.0254 -0.080236 rpy=1.5708 0 -2.0944 -> xyz=0.4064 0 -0.037489 rpy=1.5708 0 -2.0944
- joint joint_4: origin xyz=-0.30367 0.058389 0.17532 rpy=-1.5708 -0.9167 -3.1416 -> xyz=-0.303666336859734 0.0583889877211082 0.175321841329825 rpy=-1.5707963267949 -0.916697948663447 -3.14159265358979
- joint joint_5: origin xyz=-0.041507 0.086823 0.051524 rpy=0 -1.5187 -2.7485 -> xyz=-0.029571 0.071309 0.025184 rpy=0 -1.5187 -2.7485

Commit message: Added second python script.

File: ros_noetic_catkin_ws/src/full_robot_arm_urdf/urdf/full_robot_arm_urdf.urdf (robot description, URDF)
Before this commit: robot full_robot_arm_urdf, 15 links, 14 joints
Joints:
- joint base_joint: origin xyz=0.0 0.0 0.25 rpy=0 0 0 -> xyz=0.0 0.0 0.0 rpy=0 0 0
