Commit message: Fixed drivetrain hopefully.

File: drivetrain_catkin_ws/src/drivetrain_urdf/urdf/drivetrain_urdf.urdf (robot description, URDF)
Before this commit: robot drivetrain_urdf, 4 links, 3 joints
Links:
- link right_wheel: mass 0.36704 -> 0.367037154275228
Joints:
- joint left_wheel_joint: axis 0 0 0 -> 1 0 0; origin xyz=0.52793 -1.2824 0.26434 rpy=1.5708 -1.2951 3.1416 -> xyz=-0.026657 -0.33398 0.025404 rpy=0 0 0
- joint right_wheel_joint: axis 0 0 0 -> 1 0 0; origin xyz=0.52789 -0.72108 0.26435 rpy=1.5708 1.3335 -3.1416 -> xyz=0.53466 -0.33397 0.025369 rpy=0 0 0

Commit message: New Drivetrain URDF working.

File: drivetrain_catkin_ws/src/drivetrain_urdf/urdf/drivetrain_urdf.urdf (robot description, URDF)
Before this commit: robot drivetrain_urdf, 4 links, 3 joints
Joints:
- joint base_joint: origin xyz=0.0 0.0 0.0 rpy=0 0 0 -> xyz=0.0 0.0 0.02 rpy=0 0 0
