Commit message: Changed base_link to drivetrain_base_link.

File: ros_noetic_catkin_ws/src/drivetrain_urdf/urdf/drivetrain_urdf.urdf (robot description, URDF)
Before this commit: robot drivetrain_urdf, 4 links, 3 joints
Links:
- removed link base_link
- added link drivetrain_base_link, mass 18.295; collision mesh filename=package://drivetrain_urdf/meshes/drivetrain_base_link.STL; visual mesh filename=package://drivetrain_urdf/meshes/drivetrain_base_link.STL
- link right_wheel: mass 0.367037154275228 -> 0.367037154275227
Joints:
- joint base_joint: child base_link -> drivetrain_base_link
- joint left_wheel_joint: parent base_link -> drivetrain_base_link
- joint right_wheel_joint: parent base_link -> drivetrain_base_link

Commit message: Drivetrain implemented into gazebo with proper link name change.

File: ros_noetic_catkin_ws/src/drivetrain_urdf/urdf/drivetrain_urdf.urdf (robot description, URDF)
Before this commit: robot drivetrain_urdf, 4 links, 3 joints
Joints:
- removed joint base_joint
- added joint drivetrain_base_joint: type fixed, parent world, child drivetrain_base_link, origin xyz=0.0 0.0 0.05 rpy=0 0 0
