Commit message: Trying to make drivetrain work in Gazebo.

File: ros_noetic_catkin_ws/src/full_ugv_robot_urdf/urdf/full_ugv_robot_urdf.urdf (robot description, URDF)
Before this commit: robot drivetrain_urdf, 18 links, 17 joints
Links:
- removed link world
- added link root_link
- link left_wheel: geometry collision cylinder length=0.02 radius=0.0635; visual mesh filename=package://full_ugv_robot_urdf/meshes/left_wheel.STL
- link link_1: geometry collision cylinder length=0.02 radius=0.0635; visual mesh filename=package://full_ugv_robot_urdf/meshes/link_1.STL
Joints:
- joint drivetrain_base_joint: parent world -> root_link
- joint left_wheel_joint: limit (none) -> effort=5.0 velocity=10.0
- joint right_wheel_joint: limit (none) -> effort=5.0 velocity=10.0

Commit message: Working drivetrain in Gazebo using teleop keyboard.

File: ros_noetic_catkin_ws/src/full_ugv_robot_urdf/urdf/full_ugv_robot_urdf.urdf (robot description, URDF)
Before this commit: robot drivetrain_urdf, 18 links, 17 joints
Joints:
- joint left_wheel_joint: axis 1 0 0 -> -1 0 0; limit effort=5.0 velocity=10.0 -> effort=10.0 velocity=15.0
- joint right_wheel_joint: axis 1 0 0 -> -1 0 0; limit effort=5.0 velocity=10.0 -> effort=10.0 velocity=15.0

Commit message: Full Drivetrain & Arm Integration in Rviz & Gazebo

File: ros_noetic_catkin_ws/src/full_ugv_robot_urdf/urdf/full_ugv_robot_urdf.urdf (robot description, URDF)
Before this commit: robot drivetrain_urdf, 18 links, 17 joints
Joints:
- joint left_wheel_joint: limit effort=10.0 velocity=15.0 -> effort=15.0 velocity=30.0
- joint right_wheel_joint: limit effort=10.0 velocity=15.0 -> effort=15.0 velocity=30.0

Commit message: Updated full_ugv_robot_urdf.

File: ros_noetic_catkin_ws/src/full_ugv_robot_urdf/urdf/full_ugv_robot_urdf.urdf (robot description, URDF)
Before this commit: robot drivetrain_urdf, 18 links, 17 joints
Links:
- added link left_back_wheel, mass 0.36704; collision cylinder length=0.02 radius=0.0635; visual mesh filename=package://full_ugv_robot_urdf/meshes/left_back_wheel.STL
- added link left_front_wheel, mass 0.367037154275229; collision cylinder length=0.02 radius=0.0635; visual mesh filename=package://full_ugv_robot_urdf/meshes/left_front_wheel.STL
- added link right_back_wheel, mass 0; collision cylinder length=0.02 radius=0.0635; visual mesh filename=package://full_ugv_robot_urdf/meshes/right_back_wheel.STL
- added link right_front_wheel, mass 0.367037154275226; collision cylinder length=0.02 radius=0.0635; visual mesh filename=package://full_ugv_robot_urdf/meshes/right_front_wheel.STL
- link drivetrain_base_link: mass 18.295 -> 16.826
- link right_wheel: mass 0.367037154275227 -> 0.36704; geometry collision cylinder length=0.02 radius=0.0635; visual mesh filename=package://full_ugv_robot_urdf/meshes/right_wheel.STL
Joints:
- added joint left_back_wheel_joint: type continuous, parent drivetrain_base_link, child left_back_wheel, origin xyz=-0.017386 -0.56261 0.0254 rpy=0 0 0, axis -1 0 0, limit effort=15 velocity=30
- added joint left_front_wheel_joint: type continuous, parent drivetrain_base_link, child left_front_wheel, origin xyz=-0.017386 -0.10541 0.0254 rpy=0 0 0, axis -1 0 0, limit effort=15 velocity=30
- added joint right_back_wheel_joint: type continuous, parent drivetrain_base_link, child right_back_wheel, origin xyz=0.52539 -0.56261 0.0254 rpy=0 0 0, axis -1 0 0, limit effort=15 velocity=30
- added joint right_front_wheel_joint: type continuous, parent drivetrain_base_link, child right_front_wheel, origin xyz=0.52539 -0.10541 0.0254 rpy=0 0 0, axis -1 0 0, limit effort=15 velocity=30
- joint left_wheel_joint: limit effort=15.0 velocity=30.0 -> effort=15 velocity=30
- joint right_wheel_joint: limit effort=15.0 velocity=30.0 -> effort=15 velocity=30

Commit message: Reimplemented back into ROS Noetic.

File: ros_noetic_catkin_ws/src/full_ugv_robot_urdf/urdf/full_ugv_robot_urdf.urdf (robot description, URDF)
Before this commit: robot full_ugv_robot_urdf, 22 links, 21 joints
Links:
- link left_back_wheel: geometry collision cylinder length=0.02 radius=0.1; visual mesh filename=package://full_ugv_robot_urdf/meshes/left_back_wheel.STL
- link left_front_wheel: geometry collision cylinder length=0.02 radius=0.1; visual mesh filename=package://full_ugv_robot_urdf/meshes/left_front_wheel.STL
- link left_wheel: geometry collision cylinder length=0.02 radius=0.1; visual mesh filename=package://full_ugv_robot_urdf/meshes/left_wheel.STL
- link link_1: geometry collision cylinder length=0.02 radius=0.1; visual mesh filename=package://full_ugv_robot_urdf/meshes/link_1.STL
- link right_back_wheel: mass 0 -> 0.36704; geometry collision cylinder length=0.02 radius=0.1; visual mesh filename=package://full_ugv_robot_urdf/meshes/right_back_wheel.STL
- link right_front_wheel: geometry collision cylinder length=0.02 radius=0.1; visual mesh filename=package://full_ugv_robot_urdf/meshes/right_front_wheel.STL
- link right_wheel: geometry collision cylinder length=0.02 radius=0.1; visual mesh filename=package://full_ugv_robot_urdf/meshes/right_wheel.STL
