Commit message: Full integration of drivetrain & arm in ROS Gazebo.

File: ros_noetic_catkin_ws/src/full_ugv_robot_moveit_config/config/gazebo_full_ugv_robot_urdf.urdf (robot description, URDF)
Before this commit: robot drivetrain_urdf, 18 links, 17 joints
Links:
- removed link world
- added link left_back_wheel, mass 0.36704; collision cylinder length=0.02 radius=0.0635; visual mesh filename=package://full_ugv_robot_urdf/meshes/left_back_wheel.STL
- added link left_front_wheel, mass 0.367037154275229; collision cylinder length=0.02 radius=0.0635; visual mesh filename=package://full_ugv_robot_urdf/meshes/left_front_wheel.STL
- added link right_back_wheel, mass 0.36704; collision cylinder length=0.02 radius=0.0635; visual mesh filename=package://full_ugv_robot_urdf/meshes/right_back_wheel.STL
- added link right_front_wheel, mass 0.367037154275226; collision cylinder length=0.02 radius=0.0635; visual mesh filename=package://full_ugv_robot_urdf/meshes/right_front_wheel.STL
- added link root_link
- link drivetrain_base_link: mass 18.295 -> 16.826
- link left_wheel: geometry collision cylinder length=0.02 radius=0.0635; visual mesh filename=package://full_ugv_robot_urdf/meshes/left_wheel.STL
- link link_1: geometry collision cylinder length=0.02 radius=0.0635; visual mesh filename=package://full_ugv_robot_urdf/meshes/link_1.STL
- link right_wheel: mass 0.367037154275227 -> 0.36704; geometry collision cylinder length=0.02 radius=0.0635; visual mesh filename=package://full_ugv_robot_urdf/meshes/right_wheel.STL
Joints:
- added joint left_back_wheel_joint: type continuous, parent drivetrain_base_link, child left_back_wheel, origin xyz=-0.017386 -0.56261 0.0254 rpy=0 0 0, axis -1 0 0, limit effort=15 velocity=30
- added joint left_front_wheel_joint: type continuous, parent drivetrain_base_link, child left_front_wheel, origin xyz=-0.017386 -0.10541 0.0254 rpy=0 0 0, axis -1 0 0, limit effort=15 velocity=30
- added joint right_back_wheel_joint: type continuous, parent drivetrain_base_link, child right_back_wheel, origin xyz=0.52539 -0.56261 0.0254 rpy=0 0 0, axis -1 0 0, limit effort=15 velocity=30
- added joint right_front_wheel_joint: type continuous, parent drivetrain_base_link, child right_front_wheel, origin xyz=0.52539 -0.10541 0.0254 rpy=0 0 0, axis -1 0 0, limit effort=15 velocity=30
- joint drivetrain_base_joint: origin xyz=0.0 0.0 0.05 rpy=0 0 0 -> xyz=0.0 0.0 0.1 rpy=0 0 0; parent world -> root_link
- joint left_wheel_joint: axis 1 0 0 -> -1 0 0; limit (none) -> effort=15 velocity=30
- joint right_wheel_joint: axis 1 0 0 -> -1 0 0; limit (none) -> effort=15 velocity=30

File: ros_noetic_catkin_ws/src/full_ugv_robot_urdf/urdf/full_ugv_robot_urdf.urdf (robot description, URDF)
Before this commit: robot full_ugv_robot_urdf, 22 links, 21 joints
Links:
- link left_back_wheel: geometry collision cylinder length=0.02 radius=0.0635; visual mesh filename=package://full_ugv_robot_urdf/meshes/left_back_wheel.STL
- link left_front_wheel: geometry collision cylinder length=0.02 radius=0.0635; visual mesh filename=package://full_ugv_robot_urdf/meshes/left_front_wheel.STL
- link left_wheel: geometry collision cylinder length=0.02 radius=0.0635; visual mesh filename=package://full_ugv_robot_urdf/meshes/left_wheel.STL
- link link_1: geometry collision cylinder length=0.02 radius=0.0635; visual mesh filename=package://full_ugv_robot_urdf/meshes/link_1.STL
- link right_back_wheel: geometry collision cylinder length=0.02 radius=0.0635; visual mesh filename=package://full_ugv_robot_urdf/meshes/right_back_wheel.STL
- link right_front_wheel: geometry collision cylinder length=0.02 radius=0.0635; visual mesh filename=package://full_ugv_robot_urdf/meshes/right_front_wheel.STL
- link right_wheel: geometry collision cylinder length=0.02 radius=0.0635; visual mesh filename=package://full_ugv_robot_urdf/meshes/right_wheel.STL
Joints:
- joint drivetrain_base_joint: origin xyz=0.0 0.0 0.05 rpy=0 0 0 -> xyz=0.0 0.0 0.1 rpy=0 0 0
- joint left_back_wheel_joint: limit effort=15 velocity=30 -> effort=10 velocity=10
- joint left_front_wheel_joint: limit effort=15 velocity=30 -> effort=10 velocity=10
- joint left_wheel_joint: limit effort=15 velocity=30 -> effort=10 velocity=10
- joint right_back_wheel_joint: limit effort=15 velocity=30 -> effort=10 velocity=10
- joint right_front_wheel_joint: limit effort=15 velocity=30 -> effort=10 velocity=10
- joint right_wheel_joint: limit effort=15 velocity=30 -> effort=10 velocity=10
